File: dev_board.kicad_sch (KiCad schematic)
At the start: 48 parts, among them IC1 AD9609BCPZRL7-80, IC2 ENS161-BLGT_LGA9_T&R_1k5, IC3 ICM-42670-P, IC4 IWRL6432BDBAAMFR, IC5 MP4541GN-Z, IC6 THS8136IPHPR, IC7 TPS40304ADRCR, IC8 XCC1352R1F3RGZR, J2 Conn_02x26_Odd_Even, J3 Conn_02x26_Odd_Even, J4 SM03B-SRSS-TB, Q1 NMOS, Q2 NMOS, SW1 SW_Push, SW2 SW_Push, U1 RP2350_80QFN, U2 LPS22HH, Y1 ABM8-272-T3

Commit message: demarcation of boundaries, ethenret PHY
Parts:
- added U3: STM32H750VBTx, Package_QFP:LQFP-100_14x14mm_P0.5mm, symbol MCU_ST_STM32H7:STM32H750VBTx
- added U4: LAN8742A, Package_DFN_QFN:VQFN-24-1EP_4x4mm_P0.5mm_EP2.5x2.5mm_ThermalVias, symbol Interface_Ethernet:LAN8742A
Connections:
- new net: U3.10 (VSS), U3.26 (VSS), U3.49 (VSS), U3.74 (VSS), U3.99 (VSS)
Other:
- moved on the sheet: C3, C4, IC1, IC2, IC3, IC4, IC5, IC6, IC7, IC8, J2, J3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

Commit message: more pcb chanegs, ADC fixes
Parts:
- removed H1, H2, H3, H4: MountingHole, MountingHole:MountingHole_2.7mm_M2.5, symbol Mechanical:MountingHole
- removed J3: Conn_02x26_Odd_Even, Connector_PinHeader_2.54mm:PinHeader_2x26_P2.54mm_Vertical, symbol Connector_Generic:Conn_02x26_Odd_Even
- added C22, C23, C24, C26, C27, C33, C38, C41, C42, C43, C44, C45, C49, C50, C51, C52, C54, C55, C56, C57, C59, C61, C63, C66, C67, C75, C77, C82, C85, C86, C87: 100n, Capacitor_SMD:C_0402_1005Metric, symbol Device:C
- added C25, C28, C30, C31, C34, C35, C46, C53, C58, C62, C68, C70, C72, C74, C76, C83, C84: 10u, Capacitor_SMD:C_0402_1005Metric, symbol Device:C
- added C29, C32, C36, C37, C60: 1u, Capacitor_SMD:C_0402_1005Metric, symbol Device:C
- added C39, C40, C81: 10n, Capacitor_SMD:C_0402_1005Metric, symbol Device:C
- added C47, C48, C69, C71, C73, C78, C79, C80: 2.2u, Capacitor_SMD:C_0402_1005Metric, symbol Device:C
- added J5: STM32H7 GPIO/Fabric Breakout A, Connector_PinHeader_2.54mm:PinHeader_2x26_P2.54mm_Vertical, symbol Connector_Generic:Conn_02x26_Odd_Even
- added J6: STM32H7 GPIO/Fabric Breakout B, Connector_PinHeader_2.54mm:PinHeader_2x26_P2.54mm_Vertical, symbol Connector_Generic:Conn_02x26_Odd_Even
- added J9: HS/IWRL Fabric Breakout, Connector_PinHeader_2.54mm:PinHeader_2x26_P2.54mm_Vertical, symbol Connector_Generic:Conn_02x26_Odd_Even
- added L2: 10uH, Inductor_SMD:L_0805_2012Metric, symbol Device:L
- added L3: 4.7uH, Inductor_SMD:L_0805_2012Metric, symbol Device:L
- added R10, R9: 4.7k, Resistor_SMD:R_0402_1005Metric, symbol Device:R
- added R11, R12, R13, R17, R18, R19, R22, R23, R26, R27, R28, R29: 10k, Resistor_SMD:R_0402_1005Metric, symbol Device:R
- added R14: 330k, Resistor_SMD:R_0402_1005Metric, symbol Device:R
- added R15, R16: 100k, Resistor_SMD:R_0402_1005Metric, symbol Device:R
- added R20, R21, R30: 0R, Resistor_SMD:R_0402_1005Metric, symbol Device:R
- added R24: 12.1k, Resistor_SMD:R_0402_1005Metric, symbol Device:R
- added R25, R39, R40, R41: 2.2k, Resistor_SMD:R_0402_1005Metric, symbol Device:R
- added R31: 3.8k, Resistor_SMD:R_0402_1005Metric, symbol Device:R
- added R32, R33, R34, R42, R43, R44: 75, Resistor_SMD:R_0402_1005Metric, symbol Device:R
- added R35, R36, R37, R38: 49.9, Resistor_SMD:R_0402_1005Metric, symbol Device:R
Connections:
- net +1V1: now also R18.1
- net +3V3: now also IC2.4 (VDD), IC2.5 (VDDIO), IC2.7 (CSN), IC3.12 (AP_CS), IC3.5 (VDDIO), IC3.8 (VDD), IC6.40 (AVDD_2), IC6.44 (AVDD), IC8.13 (VDDS2), IC8.22 (VDDS3), IC8.34 (VDDS_DCDC), IC8.44 (VDDS), MK1.2 (VDD), U2.1 (Vdd_IO), U2.10 (VDD), U2.6 (~{CS}), U3.100 (VDD), U3.11 (VDD), U3.20 (VREF+), U3.21 (VDDA), U3.27 (VDD), U3.50 (VDD), U3.6 (VBAT), U3.75 (VDD), U4.1 (VDD2A), U4.19 (VDD1A), U4.9 (VDDIO), C22.1, C23.1, C24.1, C25.1, C26.1, C27.1, C28.1, C34.1, C35.1, C41.1, C42.1, C43.1, C44.1, C45.1, C46.1, C50.1, C51.1, C52.1, C62.1, C63.1, C80.1, C81.1, C82.1, C83.1, C84.1, C85.1, C86.1, J9.18 (Pin_18), J9.40 (Pin_40), J9.42 (Pin_42), J9.44 (Pin_44), J9.48 (Pin_48), J9.52 (Pin_52), L2.1, L3.2, R10.1, R13.1, R14.1, R17.2, R23.2, R25.2, R26.2, R28.2, R39.2, R40.2, R41.2, R9.1
- net GND: now also IC1.33 (EPAD), IC2.8 (VSS_1), IC2.9 (VSS_2), IC3.6 (GND), IC4.A1 (VSSA_1), IC4.A2 (VSSA_2), IC4.A4 (VSSA_3), IC4.A6 (VSSA_4), IC4.B2 (VSSA_5), IC4.B3 (VSSA_6), IC4.B4 (VSSA_7), IC4.B5 (VSSA_8), IC4.B6 (VSSA_9), IC4.B7 (VSS_2), IC4.C1 (VSSA_10), IC4.C2 (VSSA_11), IC4.D2 (VSSA_12), IC4.E1 (VSSA_13), IC4.E2 (VSSA_14), IC4.E5 (VSSA_PM), IC4.E6 (VSS_3), IC4.E7 (VSS_4), IC4.E8 (VSS_5), IC4.E9 (VSS_6), IC4.F2 (VSSA_15), IC4.F5 (VSSA_16), IC4.F6 (VSS_7), IC4.F7 (VSS_8), IC4.F8 (VSS_9), IC4.F9 (VSS_10), IC4.G1 (VSSA_17), IC4.G2 (VSSA_18), IC4.H12 (VSS_11), IC4.H2 (VSSA_19), IC4.J1 (VSSA_20), IC4.J2 (VSSA_21), IC4.K2 (VSSA_22), IC4.K9 (VSS_12), IC4.L1 (VSSA_23), IC4.L2 (VSSA_24), IC4.M1 (VSSA_25), IC4.M12 (VSS_13), IC4.M2 (VSSA_26), IC5.7 (GND), IC5.9 (EP), IC6.11 (DVSS), IC6.12 (DVDD), IC6.42 (AVSS_2), IC6.46 (AVSS), IC6.49 (EP), IC7.11 (GND_1), IC7.12 (GND_2), IC7.13 (GND_3), IC7.14 (GND_4), IC7.15 (GND_5), IC8.49 (EP), MK1.4 (SELECT), MK1.5 (GND), U2.3 (GND), U2.8 (GND), U2.9 (GND), U3.10 (VSS), U3.19 (VSSA), U3.26 (VSS), U3.49 (VSS), U3.74 (VSS), U3.94 (BOOT0), U3.99 (VSS), U4.25 (VSS), C22.2, C23.2, C24.2, C25.2, C26.2, C27.2, C28.2, C29.2, C30.2, C31.2, C32.2, C34.2, C35.2, C36.2, C37.2, C39.2, C40.2, C41.2, C42.2, C43.2, C44.2, C45.2, C46.2, C47.2, C48.2, C49.2, C50.2, C51.2, C52.2, C53.2, C54.2, C55.2, C56.2, C57.2, C58.2, C59.2, C60.2, C61.2, C62.2, C63.2, C66.2, C67.2, C68.2, C69.2, C70.2, C71.2, C72.2, C73.2, C74.2, C75.2, C76.2, C77.2, C78.2, C79.2, C80.2, C81.2, C82.2, C83.2, C84.2, C85.2, C86.2, C87.2, J9.17 (Pin_17), J9.38 (Pin_38), R11.2, R12.2, R15.2, R19.2, R24.2, R27.2, R29.2, R31.2, R32.2, R33.2, R34.2; no longer J2.1 (Pin_1), J2.11 (Pin_11), J2.13 (Pin_13), J2.15 (Pin_15), J2.17 (Pin_17), J2.19 (Pin_19), J2.21 (Pin_21), J2.23 (Pin_23), J2.25 (Pin_25), J2.27 (Pin_27), J2.29 (Pin_29), J2.3 (Pin_3), J2.31 (Pin_31), J2.33 (Pin_33), J2.35 (Pin_35), J2.37 (Pin_37), J2.39 (Pin_39), J2.41 (Pin_41), J2.43 (Pin_43), J2.45 (Pin_45), J2.47 (Pin_47), J2.49 (Pin_49), J2.5 (Pin_5), J2.51 (Pin_51), J2.7 (Pin_7), J2.9 (Pin_9)
- net GPIO16: now also U3.22 (PA0), J5.35 (Pin_35), J9.1 (Pin_1)
- net GPIO17: now also U3.25 (PA3), J5.38 (Pin_38), J9.2 (Pin_2)
- net GPIO18: now also U3.28 (PA4), J5.39 (Pin_39), J9.3 (Pin_3)
- net GPIO19: now also U3.29 (PA5), J5.40 (Pin_40), J9.4 (Pin_4)
- net GPIO2: now also MK1.3 (CLOCK)
- net GPIO20: now also U3.30 (PA6), J5.41 (Pin_41), J9.5 (Pin_5)
- net GPIO21: now also U3.67 (PA8), J5.43 (Pin_43), J9.6 (Pin_6)
- net GPIO22: now also U3.68 (PA9), J5.44 (Pin_44), J9.7 (Pin_7)
- net GPIO23: now also U3.69 (PA10), J5.45 (Pin_45), J9.8 (Pin_8)
- net GPIO24: now also U3.70 (PA11), J5.46 (Pin_46), J9.9 (Pin_9)
- net GPIO25: now also J2.51 (Pin_51), U3.71 (PA12), J5.47 (Pin_47), J9.10 (Pin_10)
- net GPIO26: now also J2.49 (Pin_49)
- net GPIO27: now also J2.47 (Pin_47)
- net GPIO28: now also J2.39 (Pin_39)
- net GPIO29: now also J2.37 (Pin_37)
- net GPIO3: now also MK1.1 (DATA)
- net GPIO30: now also J2.35 (Pin_35)
- net GPIO31: now also J2.33 (Pin_33)
- net GPIO32: now also IC4.A10 (QSPI_CS), J2.31 (Pin_31), U3.77 (PA15), J5.50 (Pin_50), J9.11 (Pin_11)
- net GPIO33: now also IC4.A11 (QSPI_CLK), J2.29 (Pin_29), U3.80 (PC12), J6.27 (Pin_27), J9.12 (Pin_12)
- net GPIO34: now also IC4.B11 (QSPI[0]), J2.27 (Pin_27), U3.7 (PC13), J6.28 (Pin_28), J9.13 (Pin_13)
- net GPIO35: now also IC4.B8 (QSPI[1]), J2.25 (Pin_25), U3.8 (PC14), J6.29 (Pin_29), J9.14 (Pin_14)
- net GPIO36: now also IC4.B10 (QSPI[2]), J2.23 (Pin_23), U3.9 (PC15), J6.30 (Pin_30), J9.15 (Pin_15)
- net GPIO37: now also IC4.B9 (QSPI[3]), J2.21 (Pin_21), U3.12 (PH0), J5.1 (Pin_1), J9.16 (Pin_16)
- net GPIO38: now also J2.19 (Pin_19)
- net GPIO39: now also J2.17 (Pin_17)
- net GPIO40_ADC0: now also J2.15 (Pin_15)
- net GPIO41_ADC1: now also J2.13 (Pin_13)
- net GPIO42_ADC2: now also J2.11 (Pin_11)
- net GPIO43_ADC3: now also J2.9 (Pin_9)
- net GPIO44_ADC4: now also J2.7 (Pin_7)
- net GPIO45_ADC5: now also J2.5 (Pin_5)
- net GPIO46_ADC6: now also J2.3 (Pin_3)
- net GPIO47_ADC7: now also J2.1 (Pin_1)
- net GPIO6: now also IC2.6 (INTN)
- net GPIO7: now also IC3.4 (INT1_/_INT)
- net GPIO8: now also IC3.9 (INT2)
- net GPIO9: now also U2.7 (INT_DRDY)
- net RUN: now also J2.41 (Pin_41)
- net SWCLK: now also J2.45 (Pin_45)
- net SWD: now also J2.43 (Pin_43)
- net VIN_RAW: now reaches IC7.1 (VDD)
- net VIN_RAW: now also IC5.8 (VIN), C31.1, C36.1, R16.1
- net TPS_BP: now reaches IC7.10 (BP)
- net TPS_BP: now also C37.1
- net TPS_ENSS: now reaches IC7.2 (EN/SS)
- net TPS_ENSS: now also C39.1
- net TPS_PGOOD: now reaches IC7.3 (PGOOD)
- net TPS_PGOOD: now also R17.1
- net TPS_COMP: now reaches IC7.4 (COMP)
- net TPS_COMP: now also C40.1, R22.1
- net TPS_FB: now reaches IC7.5 (FB)
- net TPS_FB: now also R18.2, R19.1, R22.2
- net TPS_BOOT: now reaches IC7.6 (BOOT)
- net TPS_BOOT: now also C38.1
- net TPS_HDRV: now reaches IC7.7 (HDRV)
- net TPS_HDRV: now also R20.1
- net TPS_SW: now reaches IC7.8 (SW)
- net TPS_SW: now also C38.2
- net TPS_LDRV_OC: now reaches IC7.9 (LDRV/_OC)
- net TPS_LDRV_OC: now also R21.1
- net ADC_CLK_P: now reaches IC1.1 (CLK+)
- net ADC_CLK_P: now also U3.44 (PE14), J5.17 (Pin_17)
- net ADC_D0: now reaches IC1.11 ((LSB)D0)
- net ADC_D0: now also U3.97 (PE0), J5.3 (Pin_3)
- net ADC_D1: now reaches IC1.12 (D1)
- net ADC_D1: now also U3.98 (PE1), J5.4 (Pin_4)
- net ADC_DRVDD: now reaches IC1.13 (DRVD0)
- net ADC_DRVDD: now also C59.1
- net ADC_D2: now reaches IC1.14 (D2)
- net ADC_D2: now also U3.1 (PE2), J5.5 (Pin_5)
- net ADC_D3: now reaches IC1.15 (D3)
- net ADC_D3: now also U3.2 (PE3), J5.6 (Pin_6)
- net ADC_D4: now reaches IC1.16 (D4)
- net ADC_D4: now also U3.3 (PE4), J5.7 (Pin_7)
- net ADC_D5: now reaches IC1.17 (D5)
- net ADC_D5: now also U3.4 (PE5), J5.8 (Pin_8)
- net ADC_D6: now reaches IC1.18 (D6)
- net ADC_D6: now also U3.5 (PE6), J5.9 (Pin_9)
- net ADC_D7: now reaches IC1.19 (D7)
- net ADC_D7: now also U3.37 (PE7), J5.10 (Pin_10)
- net ADC_CLK_N: now reaches IC1.2 (CLK-)
- net ADC_CLK_N: now also U3.45 (PE15), J5.18 (Pin_18)
- net ADC_D8: now reaches IC1.20 (D8)
- net ADC_D8: now also U3.38 (PE8), J5.11 (Pin_11)
- net ADC_D9: now reaches IC1.21 (D9(MSB))
- net ADC_D9: now also U3.39 (PE9), J5.12 (Pin_12)
- net ADC_DCO: now reaches IC1.22 (DCO)
- net ADC_DCO: now also U3.40 (PE10), J5.13 (Pin_13)
- net ADC_MODE_OR: now reaches IC1.23 (MODE/OR)
- net ADC_AVDD_1V8: now reaches IC1.24 (AVDD_4)
- net ADC_AVDD_1V8: now also IC1.29 (AVDD_3), IC1.3 (AVDD_2), IC1.32 (AVDD), C55.1, C56.1, C57.1, C58.1
- net ADC_VREF: now reaches IC1.25 (VREF)
- net ADC_VREF: now also C60.1, R30.2
- net ADC_SENSE: now reaches IC1.26 (SENSE)
- net ADC_SENSE: now also R30.1
- net ADC_VCM: now reaches IC1.27 (VCM)
- net ADC_VCM: now also C61.1
- net ADC_RBIAS: now reaches IC1.28 (RBIAS)
- net ADC_RBIAS: now also R29.1
- net ADC_VIN_N: now reaches IC1.30 (VIN-)
- net ADC_VIN_P: now reaches IC1.31 (VIN+)
- net ADC_CSB: now reaches IC1.4 (CSB)
- net ADC_CSB: now also U3.41 (PE11), J5.14 (Pin_14)
- net ADC_SCLK: now reaches IC1.5 (SCLK/DFS)
- net ADC_SCLK: now also U3.42 (PE12), J5.15 (Pin_15)
- net ADC_SDIO: now reaches IC1.6 (SDIO/PDWN)
- net ADC_SDIO: now also U3.43 (PE13), J5.16 (Pin_16)
- net SENS_I2C_SCL: now reaches U2.2 (SCL)
- net SENS_I2C_SCL: now also IC2.2 (SCLK_/_SCL), IC3.13 (AP_SCL_/_AP_SCLK), U3.92 (PB6), J6.5 (Pin_5), R9.2
- net SENS_I2C_SDA: now reaches U2.4 (SDA)
- net SENS_I2C_SDA: now also IC2.1 (MOSI_/_SDA), IC3.14 (AP_SDA_/_AP_SDIO_/_AP_SDI), U3.93 (PB7), J6.6 (Pin_6), R10.2
- net LPS_SA0: now reaches U2.5 (SA0)
- net LPS_SA0: now also R12.1
- net ENS_ADDR: now reaches IC2.3 (MISO_/_ADDR)
- net ENS_ADDR: now also R11.1
- net ETH_RXER: now reaches U4.10 (RXER/PHYAD0)
- net ETH_CRS_DV: now reaches U4.11 (CRS_DV/MODE2)
- net ETH_CRS_DV: now also U3.31 (PA7), J5.42 (Pin_42)
- net ETH_MDIO: now reaches U4.12 (MDIO)
- net ETH_MDIO: now also U3.24 (PA2), J5.37 (Pin_37), R25.1
- net ETH_MDC: now reaches U4.13 (MDC)
- net ETH_MDC: now also U3.16 (PC1), J6.16 (Pin_16)
- net ETH_REFCLK_INT: now reaches U4.14 (~{INT}/REFCLKO)
- net ETH_REFCLK_INT: now also U3.23 (PA1), J5.36 (Pin_36)
- net ETH_RST_N: now reaches U4.15 (~{RST})
- net ETH_RST_N: now also R26.1
- net ETH_TXEN: now reaches U4.16 (TXEN)
- net ETH_TXEN: now also U3.46 (PB10), J6.9 (Pin_9)
- net ETH_TXD0: now reaches U4.17 (TXD0)
- net ETH_TXD0: now also U3.51 (PB12), J6.11 (Pin_11)
- net ETH_TXD1: now reaches U4.18 (TXD1)
- net ETH_TXD1: now also U3.52 (PB13), J6.12 (Pin_12)
- net PHY_LED2_INTSEL: now reaches U4.2 (LED2/~{INTSEL})
- net PHY_LED2_INTSEL: now also R28.1
- net ETH_TX_N: now reaches U4.20 (TXN)
- net ETH_TX_N: now also R36.1
- net ETH_TX_P: now reaches U4.21 (TXP)
- net ETH_TX_P: now also R35.1
- net ETH_RX_N: now reaches U4.22 (RXN)
- net ETH_RX_N: now also R38.1
- net ETH_RX_P: now reaches U4.23 (RXP)
- net ETH_RX_P: now also R37.1
- net PHY_RBIAS: now reaches U4.24 (RBIAS)
- net PHY_RBIAS: now also R24.1
- net PHY_LED1_REGOFF: now reaches U4.3 (LED1/REGOFF)
- net PHY_LED1_REGOFF: now also R27.1
- net PHY_XTAL2: now reaches U4.4 (XTAL2)
- net PHY_XTAL1: now reaches U4.5 (XTAL1/CLKIN)
- net PHY_VDDCR: now reaches U4.6 (VDDCR)
- net PHY_VDDCR: now also C53.1, C54.1
- net ETH_RXD1: now reaches U4.7 (RXD1/MODE1)
- net ETH_RXD1: now also U3.33 (PC5), J6.20 (Pin_20)
- net ETH_RXD0: now reaches U4.8 (RXD0/MODE0)
- net ETH_RXD0: now also U3.32 (PC4), J6.19 (Pin_19)
- net IWR_TX1: now reaches IC4.A3 (TX1)
- net IWR_TX2: now reaches IC4.A5 (TX2)
- net IWR_OSC_CLK_OUT: now reaches IC4.A7 (OSC_CLK__OUT)
- net IWR_VPP: now reaches IC4.A8 (VPP)
- net IWR_CLKM: now reaches IC4.B1 (CLKM)
- net IWR_SPI_MOSI: now reaches IC4.B12 (SPIA_MOSI)
- net IWR_SPI_MOSI: now also J9.19 (Pin_19)
- net IWR_SPI_MISO: now reaches IC4.C11 (SPIA_MISO)
- net IWR_SPI_MISO: now also J9.20 (Pin_20)
- net IWR_TCK: now reaches IC4.C12 (TCK)
- net IWR_TCK: now also J9.27 (Pin_27)
- net IWR_VIO_1V8: now reaches IC4.C6 (VIOIN__18CLK)
- net IWR_VIO_1V8: now also IC4.C8 (VIOIN_18_1), IC4.G12 (VIOIN_1), IC4.K12 (VIOIN_18_2), IC4.L8 (VIOIN_18_3), IC4.M11 (VIOIN_2), IC4.M8 (VIOIN_18_4), C74.1, C75.1
- net IWR_VDD_1V2: now reaches IC4.C9 (VDD_1)
- net IWR_VDD_1V2: now also IC4.G7 (VDD_2), IC4.G8 (VDD_3), IC4.G9 (VDD_4), IC4.H8 (VDD_5), IC4.K7 (VDD_6)
- net IWR_CLKP: now reaches IC4.D1 (CLKP)
- net IWR_SPI_CLK: now reaches IC4.D10 (SPIA_CLK)
- net IWR_SPI_CLK: now also J9.21 (Pin_21)
- net IWR_SPI_CS_N: now reaches IC4.D11 (SPIA_CS0__N)
- net IWR_SPI_CS_N: now also J9.22 (Pin_22)
- net IWR_VOUT_1V4_SYNTH: now reaches IC4.D3 (VOUT__14SYNTH)
- net IWR_VOUT_1V4_SYNTH: now also C78.1
- net IWR_TDO: now reaches IC4.E11 (TDO)
- net IWR_TDO: now also J9.30 (Pin_30)
- net IWR_TMS: now reaches IC4.E12 (TMS)
- net IWR_TMS: now also J9.28 (Pin_28)
- net IWR_RX3: now reaches IC4.F1 (RX3)
- net IWR_VDDA_1V8: now reaches IC4.F3 (VDDA__18VCO)
- net IWR_VDDA_1V8: now also IC4.J5 (VIN_18PM), IC4.L5 (VDDA_18BB_1), IC4.M5 (VDDA_18BB_2), C76.1, C77.1
- net IWR_TDI: now reaches IC4.G11 (TDI)
- net IWR_TDI: now also J9.29 (Pin_29)
- net IWR_VOUT_1V4_APLL: now reaches IC4.G5 (VOUT__14APLL)
- net IWR_VOUT_1V4_APLL: now also C79.1
- net IWR_RX2: now reaches IC4.H1 (RX2)
- net IWR_GPIO_2: now reaches IC4.H10 (GPIO_2)
- net IWR_GPIO_2: now also J9.32 (Pin_32)
- net IWR_PMIC_CLKOUT: now reaches IC4.H11 (PMIC__CLKOUT)
- net IWR_PMIC_CLKOUT: now also J9.35 (Pin_35)
- net IWR_GPIO_5: now reaches IC4.J10 (GPIO_5)
- net IWR_GPIO_5: now also J9.33 (Pin_33)
- net IWR_UART_RX: now reaches IC4.J11 (UARTA_RX)
- net IWR_UART_RX: now also J9.24 (Pin_24)
- net IWR_RX1: now reaches IC4.K1 (RX1)
- net IWR_NERROR: now reaches IC4.K11 (NERROR__OUT)
- net IWR_NERROR: now also J9.31 (Pin_31)
- net IWR_NRST: now reaches IC4.L10 (NRESET)
- net IWR_NRST: now also J9.26 (Pin_26)
- net IWR_UART_RTS: now reaches IC4.L11 (UARTA_RTS)
- net IWR_UART_RTS: now also J9.25 (Pin_25)
- net IWR_UART_TX: now reaches IC4.L12 (UARTA_TX)
- net IWR_UART_TX: now also J9.23 (Pin_23)
- net IWR_VDDA_1V0RF: now reaches IC4.L3 (VDDA_10RF_1)
- net IWR_VDDA_1V0RF: now also IC4.M3 (VDDA_10RF_2), C72.1, C73.1
- net IWR_VDDA_1V2RF: now reaches IC4.L4 (VDDA_12RF_1)
- net IWR_VDDA_1V2RF: now also IC4.M4 (VDDA_12RF_2), C68.1, C69.1
- net IWR_GPADC2: now reaches IC4.L6 (GPADC2)
- net IWR_GPADC2: now also J9.37 (Pin_37)
- net IWR_HOST_CLK_REQ: now reaches IC4.M10 (HOST_CLK__REQ)
- net IWR_HOST_CLK_REQ: now also J9.34 (Pin_34)
- net IWR_GPADC1: now reaches IC4.M6 (GPADC1)
- net IWR_GPADC1: now also J9.36 (Pin_36)
- net IWR_VDD_SRAM: now reaches IC4.M7 (VDD_SRAM)
- net IWR_VDD_SRAM: now also C70.1, C71.1
- net DAC_R4: now reaches U3.13 (PH1)
- net DAC_R4: now also IC6.17 (R4), J5.2 (Pin_2)
- net STM_NRST: now reaches U3.14 (NRST)
- net STM_NRST: now also C49.1, R23.1
- net DAC_R7: now reaches U3.15 (PC0)
- net DAC_R7: now also IC6.20 (R7), J6.15 (Pin_15)
- net DAC_R8: now reaches U3.17 (PC2_C)
- net DAC_R8: now also IC6.21 (R8), J6.17 (Pin_17)
- net STM_PC3_C: now reaches U3.18 (PC3_C)
- net STM_PC3_C: now also J6.18 (Pin_18)
- net DAC_G6: now reaches U3.34 (PB0)
- net DAC_G6: now also IC6.30 (G6), J5.51 (Pin_51)
- net DAC_G7: now reaches U3.35 (PB1)
- net DAC_G7: now also IC6.29 (G7), J5.52 (Pin_52)
- net DAC_G8: now reaches U3.36 (PB2)
- net DAC_G8: now also IC6.28 (G8), J6.1 (Pin_1)
- net DAC_R9: now reaches U3.47 (PB11)
- net DAC_R9: now also IC6.22 (R9), J6.10 (Pin_10)
- net STM_VCAP1: now reaches U3.48 (VCAP)
- net STM_VCAP1: now also C47.1
- net DAC_R5: now reaches U3.53 (PB14)
- net DAC_R5: now also IC6.18 (R5), J6.13 (Pin_13)
- net DAC_R6: now reaches U3.54 (PB15)
- net DAC_R6: now also IC6.19 (R6), J6.14 (Pin_14)
- net DAC_B8: now reaches U3.55 (PD8)
- net DAC_B8: now also IC6.2 (B8), J5.27 (Pin_27)
- net DAC_B9: now reaches U3.56 (PD9)
- net DAC_B9: now also IC6.1 (B9), J5.28 (Pin_28)
- net DAC_G0: now reaches U3.57 (PD10)
- net DAC_G0: now also IC6.36 (G0), J5.29 (Pin_29)
- net DAC_G1: now reaches U3.58 (PD11)
- net DAC_G1: now also IC6.35 (G1), J5.30 (Pin_30)
- net DAC_G2: now reaches U3.59 (PD12)
- net DAC_G2: now also IC6.34 (G2), J5.31 (Pin_31)
- net DAC_G3: now reaches U3.60 (PD13)
- net DAC_G3: now also IC6.33 (G3), J5.32 (Pin_32)
- net DAC_G4: now reaches U3.61 (PD14)
- net DAC_G4: now also IC6.32 (G4), J5.33 (Pin_33)
- net DAC_G5: now reaches U3.62 (PD15)
- net DAC_G5: now also IC6.31 (G5), J5.34 (Pin_34)
- net DAC_CLK: now reaches U3.63 (PC6)
- net DAC_CLK: now also IC6.26 (CLK), J6.21 (Pin_21), R39.1
- net DAC_SYNC_T: now reaches U3.64 (PC7)
- net DAC_SYNC_T: now also IC6.25 (SYNC-T), J6.22 (Pin_22)
- net DAC_SYNC_N: now reaches U3.65 (PC8)
- net DAC_SYNC_N: now also IC6.24 (~SYNC), J6.23 (Pin_23), R41.1
- net DAC_BLANK_N: now reaches U3.66 (PC9)
- net DAC_BLANK_N: now also IC6.23 (~BLANK), J6.24 (Pin_24), R40.1
- net STM_SWDIO: now reaches U3.72 (PA13)
- net STM_SWDIO: now also J5.48 (Pin_48)
- net STM_VCAP2: now reaches U3.73 (VCAP)
- net STM_VCAP2: now also C48.1
- net STM_SWCLK: now reaches U3.76 (PA14)
- net STM_SWCLK: now also J5.49 (Pin_49)
- net DAC_M1: now reaches U3.78 (PC10)
- net DAC_M1: now also IC6.47 (M1), J6.25 (Pin_25)
- net DAC_M2: now reaches U3.79 (PC11)
- net DAC_M2: now also IC6.48 (M2), J6.26 (Pin_26)
- net DAC_B0: now reaches U3.81 (PD0)
- net DAC_B0: now also IC6.10 (B0), J5.19 (Pin_19)
- net DAC_B1: now reaches U3.82 (PD1)
- net DAC_B1: now also IC6.9 (B1), J5.20 (Pin_20)
- net DAC_B2: now reaches U3.83 (PD2)
- net DAC_B2: now also IC6.8 (B2), J5.21 (Pin_21)
- net DAC_B3: now reaches U3.84 (PD3)
- net DAC_B3: now also IC6.7 (B3), J5.22 (Pin_22)
- net DAC_B4: now reaches U3.85 (PD4)
- net DAC_B4: now also IC6.6 (B4), J5.23 (Pin_23)
- net DAC_B5: now reaches U3.86 (PD5)
- net DAC_B5: now also IC6.5 (B5), J5.24 (Pin_24)
- net DAC_B6: now reaches U3.87 (PD6)
- net DAC_B6: now also IC6.4 (B6), J5.25 (Pin_25)
- net DAC_B7: now reaches U3.88 (PD7)
- net DAC_B7: now also IC6.3 (B7), J5.26 (Pin_26)
- net DAC_G9: now reaches U3.89 (PB3)
- net DAC_G9: now also IC6.27 (G9), J6.2 (Pin_2)
- net DAC_R0: now reaches U3.90 (PB4)
- net DAC_R0: now also IC6.13 (R0), J6.3 (Pin_3)
- net DAC_R1: now reaches U3.91 (PB5)
- net DAC_R1: now also IC6.14 (R1), J6.4 (Pin_4)
- net DAC_R2: now reaches U3.95 (PB8)
- net DAC_R2: now also IC6.15 (R2), J6.7 (Pin_7)
- net DAC_R3: now reaches U3.96 (PB9)
- net DAC_R3: now also IC6.16 (R3), J6.8 (Pin_8)
- net DAC_VREF: now reaches IC6.37 (VREF)
- net DAC_VREF: now also C67.1
- net DAC_FSADJ: now reaches IC6.38 (FSADJ)
- net DAC_FSADJ: now also R31.1
- net DAC_COMP: now reaches IC6.39 (COMP)
- net DAC_COMP: now also C66.1
- net VGA_G: now reaches IC6.41 (AG)
- net VGA_G: now also R33.1, R43.1
- net VGA_R: now reaches IC6.43 (AR)
- net VGA_R: now also R32.1, R42.1
- net VGA_B: now reaches IC6.45 (AB)
- net VGA_B: now also R34.1, R44.1
- net IMU_AD0: now reaches IC3.1 (AP_SDO_/_AP_AD0)
- net IMU_FSYNC: now reaches IC3.7 (FSYNC)
- net MP_EN: now reaches IC5.1 (EN)
- net MP_EN: now also R16.2
- net MP_VCC: now reaches IC5.2 (VCC)
- net MP_VCC: now also C32.1
- net MP_FREQ: now reaches IC5.3 (FREQ)
- net MP_FB: now reaches IC5.4 (FB)
- net MP_FB: now also R14.2, R15.1
- net MP_BST: now reaches IC5.5 (BST)
- net MP_BST: now also C33.1
- net MP_SW: now reaches IC5.6 (SW)
- net MP_SW: now also C33.2, L3.1
- net CC_RF_P_2G4: now reaches IC8.1 (RF_P_2_4GHZ)
- net CC_DIO_5: now reaches IC8.10 (DIO_5)
- net CC_DIO_5: now also J6.33 (Pin_33)
- net CC_DIO_6: now reaches IC8.11 (DIO_6)
- net CC_DIO_6: now also J6.34 (Pin_34)
- net CC_DIO_7: now reaches IC8.12 (DIO_7)
- net CC_DIO_7: now also J6.35 (Pin_35)
- net CC_DIO_8: now reaches IC8.14 (DIO_8)
- net CC_DIO_8: now also J6.36 (Pin_36)
- net CC_DIO_9: now reaches IC8.15 (DIO_9)
- net CC_DIO_9: now also J6.37 (Pin_37)
- net CC_DIO_10: now reaches IC8.16 (DIO_10)
- net CC_DIO_10: now also J6.38 (Pin_38)
- net CC_DIO_11: now reaches IC8.17 (DIO_11)
- net CC_DIO_11: now also J6.39 (Pin_39)
- net CC_DIO_12: now reaches IC8.18 (DIO_12)
- net CC_DIO_12: now also J6.40 (Pin_40)
- net CC_DIO_13: now reaches IC8.19 (DIO_13)
- net CC_DIO_13: now also J6.41 (Pin_41)
- net CC_RF_N_2G4: now reaches IC8.2 (RF_N_2_4GHZ)
- net CC_DIO_14: now reaches IC8.20 (DIO_14)
- net CC_DIO_14: now also J6.42 (Pin_42)
- net CC_DIO_15: now reaches IC8.21 (DIO_15)
- net CC_DIO_15: now also J6.43 (Pin_43)
- net CC_DCOUPL: now reaches IC8.23 (DCOUPL)
- net CC_DCOUPL: now also C29.1
- net CC_TMSC: now reaches IC8.24 (JTAG_TMSC)
- net CC_TMSC: now also J9.50 (Pin_50)
- net CC_TCKC: now reaches IC8.25 (JTAG_TCKC)
- net CC_TCKC: now also J6.45 (Pin_45)
- net CC_DIO_16: now reaches IC8.26 (DIO_16)
- net CC_DIO_16: now also J6.44 (Pin_44)
- net CC_DIO_17: now reaches IC8.27 (DIO_17)
- net CC_DIO_17: now also J9.39 (Pin_39)
- net CC_DIO_18: now reaches IC8.28 (DIO_18)
- net CC_DIO_18: now also J6.46 (Pin_46)
- net CC_DIO_19: now reaches IC8.29 (DIO_19)
- net CC_DIO_19: now also J9.41 (Pin_41)
- net CC_RF_P_SUBG: now reaches IC8.3 (RF_P_SUB_1GHZ)
- net CC_DIO_20: now reaches IC8.30 (DIO_20)
- net CC_DIO_20: now also J6.48 (Pin_48)
- net CC_DIO_21: now reaches IC8.31 (DIO_21)
- net CC_DIO_21: now also J9.43 (Pin_43)
- net CC_DIO_22: now reaches IC8.32 (DIO_22)
- net CC_DIO_22: now also J6.50 (Pin_50)
- net CC_DCDC_SW: now reaches IC8.33 (DCDC_SW)
- net CC_DCDC_SW: now also L2.2
- net CC_RESET_N: now reaches IC8.35 (RESET_N)
- net CC_RESET_N: now also J9.46 (Pin_46), R13.2
- net CC_DIO_23: now reaches IC8.36 (DIO_23)
- net CC_DIO_23: now also J9.45 (Pin_45)
- net CC_DIO_24: now reaches IC8.37 (DIO_24)
- net CC_DIO_24: now also J6.52 (Pin_52)
- net CC_DIO_25: now reaches IC8.38 (DIO_25)
- net CC_DIO_25: now also J9.47 (Pin_47)
- net CC_DIO_26: now reaches IC8.39 (DIO_26)
- net CC_DIO_26: now also J6.51 (Pin_51)
- net CC_RF_N_SUBG: now reaches IC8.4 (RF_N_SUB_1GHZ)
- net CC_DIO_27: now reaches IC8.40 (DIO_27)
- net CC_DIO_27: now also J9.49 (Pin_49)
- net CC_DIO_28: now reaches IC8.41 (DIO_28)
- net CC_DIO_28: now also J6.49 (Pin_49)
- net CC_DIO_29: now reaches IC8.42 (DIO_29)
- net CC_DIO_29: now also J9.51 (Pin_51)
- net CC_DIO_30: now reaches IC8.43 (DIO_30)
- net CC_DIO_30: now also J6.47 (Pin_47)
- net CC_VDDR: now reaches IC8.45 (VDDR)
- net CC_VDDR: now also IC8.48 (VDDR_RF), C30.1
- net CC_X48M_N: now reaches IC8.46 (X48M_N)
- net CC_X48M_P: now reaches IC8.47 (X48M_P)
- net CC_X32K_Q1: now reaches IC8.6 (X32K_Q1)
- net CC_X32K_Q2: now reaches IC8.7 (X32K_Q2)
- net CC_DIO_3: now reaches IC8.8 (DIO_3)
- net CC_DIO_3: now also J6.31 (Pin_31)
- net CC_DIO_4: now reaches IC8.9 (DIO_4)
- net CC_DIO_4: now also J6.32 (Pin_32)
- new net ETH_CT: C87.1, R35.2, R36.2, R37.2, R38.2
- new net Q1_GATE: R20.2
- new net Q2_GATE: R21.2
- new net VGA_MON: R42.2, R43.2, R44.2
Other:
- note added: "ADC and THS8136 analog support below boundary"
- note added: "ADC island: AD9609 AVDD/DRVDD/VREF/VCM/RBIAS support"
- note added: "ADC island: PE0-PE15 assigned to AD9609 data/control/clock nets"
- note added: "ADC/THS8136: digital buses are named for routing clarity; analog inputs/outputs need final connector or front-end choice."
- note added: "Boot/strap pins are tied by labels and pull resistors; change these only with firmware/boot-mode review."
- note added: "Buck regulator recommended bootstrap, feedback, soft-start and compensation parts"
- note added: "CC1352 island: DCOUPL/VDDR/DCDC/crystal support"
- note added: "CC1352 island: recommended decoupling, DCDC and crystal nets"
- note added: "CC1352: DCOUPL/VDDR/DCDC support is shown; RF balun/matching network should follow the selected reference design."
- note added: "Codex generated recommended support components - cross-boundary data uses labels only"
- note added: "DAC island: PD/PB/PC/PH1 assigned to THS8136 RGB bus/timing; fabric is kept off these pins."
- note added: "DAC island: THS8136 DVDD/AVDD/VREF/FSADJ/output loads"
- note added: "Electrical net names preserve existing RP2350 GPIO labels; role notes map those GPIOs to HS_Dx/QSPI functions."
- note added: "Ethernet island: LAN8742A RBIAS, VDDCR, magnetics termination"
- note added: "Extra explicit passives from datasheet application/BOM sections"
- note added: "Fabric island: GPIO32=CS, GPIO33=CLK, GPIO34-37=IO0-IO3"
- note added: "Fabric island: high-speed hub and combined GPIO/IWRL breakout fabric"
- note added: "I2C sensor bus: ENS161, ICM-42670-P, and LPS22HH share SENS_I2C_SCL/SDA with 4.7k pullups."
- note added: "IWRL island: LDO-output 10u + 2.2u capacitors"
- note added: "IWRL island: LDO-output and supply decoupling below boundary"
- note added: "IWRL6432: LDO-output caps follow datasheet typical 10u + 2.2u groups; RF pins still need layout/reference-design matching."
- note added: "Intentional crossings: GPIO16-GPIO25 are RP-to-STM parallel fabric; GPIO32-GPIO37 are shared RP/STM/IWR QSPI."
- note added: "Island plan: PE=ADC, PD/PB/PC/PH1=DAC, PA+PC12-15+PH0=fabric, Ethernet keeps existing PA/PB/PC pins."
- note added: "J9 combines the fabric and IWRL breakout: GPIO32-37 are the IWRL high-speed QSPI bus; lower pins expose IWRL SPIA/UART/JTAG/control."
- note added: "Keep exact/application-specific values for PHY RBIAS 12.1k, Ethernet 49.9R, video 75R, DAC FSADJ 3.8k."
- note added: "No generated data wire crosses the horizontal user boundary; shared signals use local net labels."
- note added: "Power island: buck bootstrap, comp, feedback, SS and FET gate resistors"
- note added: "Power rails: labels mark intended rails; add PWR_FLAGs after final regulator/connector source choices."
- note added: "RP-to-STM parallel fabric: GPIO16-23=HS_D0-D7, GPIO24=HS_CLK, GPIO25=HS_FRAME"
- note added: "Review before layout: RF matching, ADC analog front-end, Ethernet magnetics, and regulator loop values are topology-dependent."
- note added: "STM32 island: VDD/VDDA/VCAP decoupling"
- note added: "STM32/LAN8742A: RMII nets are label-connected below the boundary; unused STM32 GPIOs are intentionally left for expansion."
- note added: "STM32H750 and LAN8742A support below boundary"
- note added: "Schematic completion notes"
- note added: "Sensor I2C pulls and local decoupling"
- note added: "Value consolidation: generic passives use 100n, 1u, 2.2u, 10u, 10n, 10k, 100k, 2.2k where practical."
- moved on the sheet: IC1, IC4, IC5, IC6, IC7, MK1, Q1, Q2, U2, U4

Commit message: more pcb chanegs, placements
Parts:
- removed Q1, Q2: NMOS, Package_SON:Infineon_PG-TDSON-8_6.15x5.15mm, symbol Simulation_SPICE:NMOS
- added C88, C90, C92, C93, C94: 100n, Capacitor_SMD:C_0402_1005Metric, symbol Device:C
- added C89: 1n, Capacitor_SMD:C_0402_1005Metric, symbol Device:C
- added C91: 22p, Capacitor_SMD:C_0402_1005Metric, symbol Device:C
- added J10: RJ45 / 8P8C LED, Connector_RJ:RJ45_Amphenol_RJMG1BD3B8K1ANR, symbol Connector:8P8C_LED_Shielded
- added J11: SMA_RF_LAUNCH, Connector_Coaxial:SMA_Amphenol_132134-10_Vertical, symbol Connector:Conn_Coaxial
- added J12: RP2350 USB PROGRAM, Connector_USB:USB_Micro-B_Amphenol_10103594-0001LF_Horizontal, symbol Connector:USB_B_Micro
- added J13: STM32 USB DFU ALT, Connector_USB:USB_Micro-B_Amphenol_10103594-0001LF_Horizontal, symbol Connector:USB_B_Micro
- added J14: CC1352 PROG BRIDGE USB, Connector_USB:USB_Micro-B_Amphenol_10103594-0001LF_Horizontal, symbol Connector:USB_B_Micro
- added J15: IWRL USB PROGRAM, Connector_USB:USB_Micro-B_Amphenol_10103594-0001LF_Horizontal, symbol Connector:USB_B_Micro
- added R45, R46, R47, R48: 1k, Resistor_SMD:R_0402_1005Metric, symbol Device:R
- added R49, R50: 33, Resistor_SMD:R_0402_1005Metric, symbol Device:R
- added R51: 0R/DNP, Resistor_SMD:R_0402_1005Metric, symbol Device:R
- added TP1, TP2: TestPoint, TestPoint:TestPoint_Pad_3.0x3.0mm, symbol Connector:TestPoint
- added U5: PGA113, Package_SO:TSSOP-10_3x3mm_P0.5mm, symbol Analog:PGA113
- added U6: MCP6D11T-E/MS, MCP6D11T:MCP6D11T-E_MSOP-8_3x3mm_P0.65mm, symbol MCP6D11T:MCP6D11T-E_MS
- added U7: FT232RNL-TUBE, Package_SO:SSOP-28_5.3x10.2mm_P0.65mm, symbol Interface_USB:FT232RL
Connections:
- net GPIO27 is gone; now on net CC_DIO_6: J2.47 (Pin_47), U1.28 (GPIO27)
- net GPIO28 is gone; now on net CC_DIO_7: J2.39 (Pin_39), U1.36 (GPIO28)
- net GPIO29 is gone; now on net CC_DIO_8: J2.37 (Pin_37), U1.37 (GPIO29)
- net GPIO30 is gone; now on net CC_DIO_9: J2.35 (Pin_35), U1.38 (GPIO30)
- net GPIO31 is gone; now on net CC_DIO_10: J2.33 (Pin_33), U1.39 (GPIO31)
- net IMU_FSYNC is gone; now on net +3V3: IC3.7 (FSYNC)
- net +3V3: now also MK1.5 (GND), C88.2, C89.2, C90.2, R46.2, R47.1, R47.2, R50.1, U5.1 (AV_{DD}), U5.10 (DV_{DD}), U6.1 (IN-), U6.3 (VDD), U6.4 (OUT+); no longer IC2.7 (CSN), MK1.2 (VDD)
- net ADC_VCM: now also R46.1, U5.4 (V_{REF}), U6.2 (VOCM)
- net ADC_VIN_N: now also C91.2, R49.2
- net ADC_VIN_P: now also C91.1, R50.2
- net ETH_RX_N: now also J10.6 (RD-)
- net ETH_RX_P: now also J10.3 (RD+)
- net ETH_TX_N: now also J10.2 (TD-)
- net ETH_TX_P: now also J10.1 (TD+)
- net GND: now also MK1.2 (VDD), C88.1, C89.1, C90.1, C92.2, C93.2, C94.2, J10.13 (Shield), J12.5 (GND), J12.6 (Shield), J13.5 (GND), J13.6 (Shield), J14.5 (GND), J14.6 (Shield), J15.5 (GND), J15.6 (Shield), U5.6 (GND), U6.6 (VSS), U7.18 (GND), U7.21 (GND), U7.25 (AGND), U7.26 (TEST), U7.7 (GND); no longer MK1.4 (SELECT), MK1.5 (GND)
- net GPIO10: now also U5.7 (SCLK)
- net GPIO11: now also U5.8 (DIO)
- net GPIO12: now also U5.9 (~{CS})
- net GPIO13: now also U6.7 (~PD)
- net GPIO3: now also MK1.4 (SELECT); no longer MK1.1 (DATA)
- net GPIO37: no longer U3.12 (PH0)
- net GPIO4: now also MK1.1 (DATA)
- net GPIO6: now also IC2.7 (CSN); no longer IC2.6 (INTN)
- net GPIO8: no longer IC3.9 (INT2)
- net IWR_UART_RX: now also U7.1 (TXD)
- net IWR_UART_TX: now also U7.5 (RXD)
- net IWR_VIO_1V8: now also C93.1, U7.19 (~{RESET}), U7.4 (VCCIO)
- net PHY_LED1_REGOFF: now also J10.9 (LED1A)
- net PHY_LED2_INTSEL: now also J10.11 (LED2A)
- net USB_D+: now also J12.3 (D+)
- net USB_D-: now also J12.2 (D-)
- net VIN_RAW: now also J12.1 (VBUS), J14.1 (VBUS)
- new net: R48.2, R49.1, U6.5 (OUT-)
- new net: R45.2, R48.1, U6.8 (IN+)
- new net: R45.1, U5.5 (V_{OUT})
- new net CC_PROG_USB_D+: J14.3 (D+)
- new net CC_PROG_USB_D-: J14.2 (D-)
- new net CC_PROG_USB_VBUS: J14.4 (ID)
- new net ETH_CT1: J10.5 (CT2)
- new net ETH_CT2: J10.4 (CT1)
- new net IWR_FTDI_3V3OUT: C94.1, U7.17 (3V3OUT)
- new net IWR_PROG_USB_D+: J15.3 (D+), U7.15 (USBD+)
- new net IWR_PROG_USB_D-: J15.2 (D-), U7.16 (USBD-)
- new net IWR_USB_VBUS: C92.1, J15.1 (VBUS), U7.20 (VCC)
- new net SCOPE_AUX_IN: TP2.1, U5.2 (CH1)
- new net SCOPE_IN: TP1.1, U5.3 (CH0/V_{CAL})
- new net STM_USB_FS_DM: J13.2 (D-)
- new net STM_USB_FS_DP: J13.3 (D+)
- new net STM_USB_VBUS: J13.1 (VBUS)
- new net STM_VCAP_A: U3.12 (PH0)
- no-connect marks 0 -> 14
Other:
- note added: "CC1352 has no native USB device port; J14 is the USB side of an XDS110/cJTAG bridge to CC_TMSC, CC_TCKC, and CC_RESET_N."
- note added: "Place 1k FDA gain/feedback resistors tight to MCP6D11 pins; place 33R/22p ADC filter tight to AD9609 VIN pins."
- note added: "RF SMA launch: stuff after selected CC1352 balun/matching network; keep 50 ohm controlled impedance."
- note added: "RF connector is a configurable launch; review CC1352 reference matching before populating R51."
- note added: "RJ45 Ethernet island: cable connector / MagJack-side breakout for LAN8742A pairs and LEDs."
- note added: "RP2350 scope control: GPIO10=PGA SCLK, GPIO11=PGA SDIO, GPIO12=PGA CS_N, GPIO13=MCP6D11 PD_N"
- note added: "STM32 DFU uses PA11/PA12; R52/R53 are DNP because those pins are currently assigned to RMII Ethernet nets."
- note added: "Scope ADC front-end: single-ended input, PGA113 gain, MCP6D11 differential ADC driver"
- note added: "USB programming ports: J12 RP2350 native USB; J13 STM32 DFU optional via R52/R53; J14 CC1352 programmer bridge USB input; J15 IWRL USB-UART at 1.8V I/O."
- moved on the sheet: U2, U4

Commit message: more fixes
Parts:
- removed R20, R21: 0R, Resistor_SMD:R_0402_1005Metric, symbol Device:R
Connections:
- net +3V3: no longer C89.2, C90.2, R46.2, R47.1, R47.2, R50.1, U6.1 (IN-), U6.4 (OUT+)
- new net: C90.2, R47.2, R50.1, U6.4 (OUT+)
- new net: C89.2, R46.2, R47.1, U6.1 (IN-)
Other:
- moved on the sheet: C92, C93, C94, R47

Commit message: more fixes
Parts:
- added IC10: MP4541GN-Z, SOIC127P600X170-9N, symbol MP4541GN-Z:MP4541GN-Z
- added IC9: TPS40304ADRCR, TPS40304ADRCR, symbol TPS40304ADRCR:TPS40304ADRCR
- added TP3, TP4, TP5: TestPoint, TestPoint:TestPoint_Pad_3.0x3.0mm, symbol Connector:TestPoint
Connections:
- net +3V3: no longer J9.42 (Pin_42), J9.48 (Pin_48)
- net GND: now also J9.42 (Pin_42), J9.48 (Pin_48), IC10.7 (GND), IC10.9 (EP), IC9.11 (GND_1), IC9.12 (GND_2), IC9.13 (GND_3), IC9.14 (GND_4), IC9.15 (GND_5)
- net MP_BST: now also IC10.5 (BST)
- net MP_EN: now also IC10.1 (EN)
- net MP_FB: now also IC10.4 (FB)
- net MP_FREQ: now also IC10.3 (FREQ)
- net MP_SW: now also IC10.6 (SW)
- net MP_VCC: now also IC10.2 (VCC)
- net TPS_BOOT: now also IC9.6 (BOOT)
- net TPS_BP: now also IC9.10 (BP)
- net TPS_COMP: now also IC9.4 (COMP)
- net TPS_ENSS: now also IC9.2 (EN/SS)
- net TPS_FB: now also IC9.5 (FB)
- net TPS_HDRV: now also IC9.7 (HDRV)
- net TPS_LDRV_OC: now also IC9.9 (LDRV/_OC)
- net TPS_PGOOD: now also IC9.3 (PGOOD)
- net TPS_SW: now also IC9.8 (SW)
- net VGA_B: now also TP4.1
- net VGA_G: now also TP5.1
- net VGA_R: now also TP3.1
- net VIN_RAW: now also IC10.8 (VIN), IC9.1 (VDD)

Commit message: more fixes
Changed lines of the file:
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@@
+	(symbol
+		(lib_id "power:GND")
+		(at 763.27 565.15 0)
+		(unit 1)
+		(exclude_from_sim no)
+		(in_bom yes)
+		(on_board yes)
+		(dnp no)
+		(property "Reference" "#PWR999"
+			(at 763.27 571.5 0)
+			(effects
+				(font
+					(size 1.27 1.27)
+				)
+				(hide yes)
+			)
+		)
+		(property "Value" "GND"
+			(at 763.397 569.5442 0)
+			(effects
+				(font
+					(size 1.27 1.27)
+				)
+			)
+		)
+		(property "Footprint" ""
+			(at 763.27 565.15 0)
+			(effects
+				(font
+					(size 1.27 1.27)
+				)
+				(hide yes)
+			)
+		)
+		(property "Datasheet" ""
+			(at 763.27 565.15 0)
+			(effects
+				(font
+					(size 1.27 1.27)
+				)
+				(hide yes)
+			)
+		)
+		(property "Description" ""
+			(at 763.27 565.15 0)
+			(effects
+				(font
+					(size 1.27 1.27)
+				)
+			)
+		)
+		(pin "1"
+		)
+		(instances
+			(project ""
+				(path "/94683f5c-9cd9-448e-be96-9792537b5cb8"
+					(reference "#PWR999")
+					(unit 1)
+				)
+			)
+		)
+	)
+	(wire
+		(pts
+			(xy 758.19 565.15) (xy 763.27 565.15)
+		)
+		(stroke
+			(width 0)
+			(type default)
+		)
+	)
 	(symbol
 		(lib_id "power:GND")

Commit message: more fixes
Other:
- note added: "I2C sensor bus: ENS161, ICM-42670-P, and LPS22HH share SENS_I2C_SCL/SDA with one pullup pair; strap ENS_ADDR, IMU_AD0, and LPS_SA0 intentionally."
- note removed: "I2C sensor bus: ENS161, ICM-42670-P, and LPS22HH share SENS_I2C_SCL/SDA with 4.7k pullups."
Changed lines of the file:
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@@
 		)
 	)
-	(text "I2C sensor bus: ENS161, ICM-42670-P, and LPS22HH share SENS_I2C_SCL/SDA with 4.7k pullups."
+	(text "I2C sensor bus: ENS161, ICM-42670-P, and LPS22HH share SENS_I2C_SCL/SDA with one pullup pair; strap ENS_ADDR, IMU_AD0, and LPS_SA0 intentionally."
 		(exclude_from_sim no)
 		(at 518.16 212.09 0)
