File: dev_board.kicad_sch (KiCad schematic)
At the start: 176 parts, among them IC1 AD9609BCPZRL7-80, IC10 MP4541GN-Z, IC2 ENS161-BLGT_LGA9_T&R_1k5, IC3 ICM-42670-P, IC4 IWRL6432BDBAAMFR, IC5 MP4541GN-Z, IC6 THS8136IPHPR, IC7 TPS40304ADRCR, IC8 XCC1352R1F3RGZR, IC9 TPS40304ADRCR, J10 RJ45 / 8P8C LED, J11 SMA_RF_LAUNCH, J12 RP2350 USB PROGRAM, J13 STM32 USB DFU ALT, J14 CC1352 PROG BRIDGE USB, J15 IWRL USB PROGRAM, J2 Conn_02x26_Odd_Even, J4 SM03B-SRSS-TB, J5 STM32H7 GPIO/Fabric Breakout A, J6 STM32H7 GPIO/Fabric Breakout B, J9 HS/IWRL Fabric Breakout, SW1 SW_Push, SW2 SW_Push, U1 RP2350_80QFN, U2 LPS22HH, U3 STM32H750VBTx, U4 LAN8742A, U5 PGA113, U6 MCP6D11T-E/MS, U7 FT232RNL-TUBE, Y1 ABM8-272-T3

Commit message: something
Parts:
- added C95: 47n, Capacitor_SMD:C_0402_1005Metric, symbol Device:C
- C3: now not fitted
- J13: value STM32 USB DFU ALT -> DNP / not used
- J14: value CC1352 PROG BRIDGE USB -> DNP / not used
Connections:
- net VREG_LX is gone; now on net RP_SWCLK: L1.2, U1.63 (VREG_LX)
- net +1V1: now also J2.43 (Pin_43), J4.3 (Pin_3)
- net SWCLK renamed RP_SWCLK
- removed net SWD: J2.43 (Pin_43), J4.3 (Pin_3), U1.34 (SWD)
- new net VREG_FB: U1.34 (SWD)
- no-connect marks 14 -> 15
Other:
- note added: "CC1352 has no native USB device port; J14 is the USB side of an XDS110/cJTAG bridge to CC_TMSC, CC_TCKC, and CC_RESET_N, but is DNP in this revision."
- note added: "I2C sensor bus: ENS161, ICM-42670-P, and LPS22HH share SENS_I2C_SCL/SDA with one pullup pair; strap ENS_ADDR, IMU_AD0, and LPS_SA0 intentionally; IC2 INTN -> GPIO27 and IC3 INT2 -> GPIO28."
- note added: "USB programming ports: J12 RP2350 native USB; J13 STM32 DFU optional via R52/R53; J14 CC1352 programmer bridge USB input, DNP in this revision; J15 IWRL USB-UART at 1.8V I/O."
- note removed: "CC1352 has no native USB device port; J14 is the USB side of an XDS110/cJTAG bridge to CC_TMSC, CC_TCKC, and CC_RESET_N."
- note removed: "I2C sensor bus: ENS161, ICM-42670-P, and LPS22HH share SENS_I2C_SCL/SDA with one pullup pair; strap ENS_ADDR, IMU_AD0, and LPS_SA0 intentionally."
- note removed: "USB programming ports: J12 RP2350 native USB; J13 STM32 DFU optional via R52/R53; J14 CC1352 programmer bridge USB input; J15 IWRL USB-UART at 1.8V I/O."
Changed lines of the file:
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@@
 		)
 	)
-	(text "USB programming ports: J12 RP2350 native USB; J13 STM32 DFU optional via R52/R53; J14 CC1352 programmer bridge USB input; J15 IWRL USB-UART at 1.8V I/O."
+	(text "USB programming ports: J12 RP2350 native USB; J13 STM32 DFU optional via R52/R53; J14 CC1352 programmer bridge USB input, DNP in this revision; J15 IWRL USB-UART at 1.8V I/O."
 		(exclude_from_sim no)
 		(at 797.56 76.454 0)
@@
 		)
 	)
-	(text "I2C sensor bus: ENS161, ICM-42670-P, and LPS22HH share SENS_I2C_SCL/SDA with one pullup pair; strap ENS_ADDR, IMU_AD0, and LPS_SA0 intentionally."
+	(text "I2C sensor bus: ENS161, ICM-42670-P, and LPS22HH share SENS_I2C_SCL/SDA with one pullup pair; strap ENS_ADDR, IMU_AD0, and LPS_SA0 intentionally; IC2 INTN -> GPIO27 and IC3 INT2 -> GPIO28."
 		(exclude_from_sim no)
 		(at 518.16 212.09 0)
@@
 		)
 	)
-	(text "CC1352 has no native USB device port; J14 is the USB side of an XDS110/cJTAG bridge to CC_TMSC, CC_TCKC, and CC_RESET_N."
+	(text "CC1352 has no native USB device port; J14 is the USB side of an XDS110/cJTAG bridge to CC_TMSC, CC_TCKC, and CC_RESET_N, but is DNP in this revision."
 		(exclude_from_sim no)
 		(at 792.22 177.54 0)
@@
 	(wire
 		(pts
+			(xy 758.19 565.15) (xy 763.27 565.15)
+		)
+		(stroke
+			(width 0)
+			(type default)
+		)
+	)
+	(wire
+		(pts
 			(xy 100.33 599.44) (xy 91.44 599.44)
 		)
@@
 		)
 	)
-	(label "SWCLK"
+	(label "RP_SWCLK"
 		(at 325.12 154.94 0)
 		(effects
@@
 		)
 	)
-	(label "SWD"
+	(label "RP_SWDIO"
 		(at 318.77 189.23 0)
 		(effects
@@
 		)
 	)
-	(label "SWCLK"
+	(label "VREG_LX"
 		(at 152.4 176.53 0)
 		(effects
@@
 		)
 	)
-	(label "SWD"
+	(label "RP_SWDIO"
 		(at 325.12 152.4 0)
 		(effects
@@
 		)
 	)
+	(label "RP_SWCLK"
+		(at 134.62 113.03 0)
+		(effects
+			(font
+				(size 1.27 1.27)
+			)
+			(justify left bottom)
+		)
+	)
+	(label "RP_SWDIO"
+		(at 142.24 110.49 0)
+		(effects
+			(font
+				(size 1.27 1.27)
+			)
+			(justify left bottom)
+		)
+	)
 	(label "GND"
 		(at 810.26 389.89 0)
@@
 		)
 	)
-	(label "SWCLK"
+	(label "RP_SWCLK"
 		(at 318.77 184.15 0)
 		(effects
@@
 		)
 	)
-	(label "SWD"
+	(label "VREG_FB"
 		(at 152.4 179.07 0)
 		(effects
@@
 		(in_bom yes)
 		(on_board yes)
-		(dnp no)
+		(dnp yes)
 		(property "Reference" "C3"
 			(at 366.9284 187.071 0)
@@
 	(symbol
 		(lib_id "power:GND")
-		(at 763.27 565.15 0)
-		(unit 1)
-		(exclude_from_sim no)
-		(in_bom yes)
-		(on_board yes)
-		(dnp no)
-		(property "Reference" "#PWR999"
-			(at 763.27 571.5 0)
-			(effects
-				(font
-					(size 1.27 1.27)
-				)
-				(hide yes)
-			)
-		)
-		(property "Value" "GND"
-			(at 763.397 569.5442 0)
-			(effects
-				(font
-					(size 1.27 1.27)
-				)
-			)
-		)
-		(property "Footprint" ""
-			(at 763.27 565.15 0)
-			(effects
-				(font
-					(size 1.27 1.27)
-				)
-				(hide yes)
-			)
-		)
-		(property "Datasheet" ""
-			(at 763.27 565.15 0)
-			(effects
-				(font
-					(size 1.27 1.27)
-				)
-				(hide yes)
-			)
-		)
-		(property "Description" ""
-			(at 763.27 565.15 0)
-			(effects
-				(font
-					(size 1.27 1.27)
-				)
-			)
-		)
-		(pin "1"
-		)
-		(instances
-			(project ""
-				(path "/94683f5c-9cd9-448e-be96-9792537b5cb8"
-					(reference "#PWR999")
-					(unit 1)
-				)
-			)
-		)
-	)
-	(wire
-		(pts
-			(xy 758.19 565.15) (xy 763.27 565.15)
-		)
-		(stroke
-			(width 0)
-			(type default)
-		)
-	)
-	(symbol
-		(lib_id "power:GND")
 		(at 143.51 73.66 0)
 		(unit 1)
@@
 			)
 		)
-		(property "Value" "CC1352 PROG BRIDGE USB"
+		(property "Value" "DNP / not used"
 			(at 801.37 149.86 0)
 			(effects
@@
 	)
 	(symbol
+		(lib_id "power:GND")
+		(at 763.27 565.15 0)
+		(unit 1)
+		(exclude_from_sim no)
+		(in_bom yes)
+		(on_board yes)
+		(dnp yes)
+		(property "Reference" "#PWR999"
+			(at 763.27 571.5 0)
+			(effects
+				(font
+					(size 1.27 1.27)
+				)
+				(hide yes)
+			)
+		)
+		(property "Value" "GND"
+			(at 763.397 569.5442 0)
+			(effects
+				(font
+					(size 1.27 1.27)
+				)
+			)
+		)
+		(property "Footprint" ""
+			(at 763.27 565.15 0)
+			(effects
+				(font
+					(size 1.27 1.27)
+				)
+				(hide yes)
+			)
+		)
+		(property "Datasheet" ""
+			(at 763.27 565.15 0)
+			(effects
+				(font
+					(size 1.27 1.27)
+				)
+				(hide yes)
+			)
+		)
+		(property "Description" ""
+			(at 763.27 565.15 0)
+			(effects
+				(font
+					(size 1.27 1.27)
+				)
+			)
+		)
+		(pin "1"
+		)
+		(instances
+			(project ""
+				(path "/94683f5c-9cd9-448e-be96-9792537b5cb8"
+					(reference "#PWR999")
+					(unit 1)
+				)
+			)
+		)
+	)
+	(symbol
 		(lib_id "Device:R")
 		(at 354.33 427.99 90)
@@
 			)
 		)
-		(property "Value" "STM32 USB DFU ALT"
+		(property "Value" "DNP / not used"
 			(at 807.72 119.38 0)
 			(effects
@@
 		)
 	)
+	(symbol
+		(lib_id "Device:C")
+		(at 690 565.15 90)
+		(unit 1)
+		(exclude_from_sim no)
+		(in_bom yes)
+		(on_board yes)
+		(dnp no)
+		(property "Reference" "C95"
+			(at 691.27 563.88 0)
+			(effects
+				(font
+					(size 1.27 1.27)
+				)
+			)
+		)
+		(property "Value" "47n"
+			(at 691.27 566.42 0)
+			(effects
+				(font
+					(size 1.27 1.27)
+				)
+			)
+		)
+		(property "Footprint" "Capacitor_SMD:C_0402_1005Metric"
+			(at 690 568.96 90)
+			(effects
+				(font
+					(size 1.27 1.27)
+				)
+				(hide yes)
+			)
+		)
+		(property "Datasheet" "~"
+			(at 690 568.96 90)
+			(effects
+				(font
+					(size 1.27 1.27)
+				)
+				(hide yes)
+			)
+		)
+		(property "Description" "IWRL6432 VBGAP decoupling capacitor"
+			(at 690 565.15 90)
+			(effects
+				(font
+					(size 1.27 1.27)
+				)
+			)
+		)
+		(pin "1"
+		)
+		(pin "2"
+		)
+		(instances
+			(project ""
+				(path "/94683f5c-9cd9-448e-be96-9792537b5cb8"
+					(reference "C95")
+					(unit 1)
+				)
+			)
+		)
+	)
+	(wire
+		(pts
+			(xy 414.02 406.4) (xy 421.64 406.4)
+		)
+		(stroke
+			(width 0)
+			(type default)
+		)
+	)
+	(label "+3V3"
+		(at 421.64 406.4 0)
+		(effects
+			(font
+				(size 1.27 1.27)
+			)
+			(justify left bottom)
+		)
+	)
+	(wire
+		(pts
+			(xy 758.19 565.15) (xy 758.19 560.07)
+		)
+		(stroke
+			(width 0)
+			(type default)
+		)
+	)
+	(label "GND"
+		(at 758.19 560.07 0)
+		(effects
+			(font
+				(size 1.27 1.27)
+			)
+			(justify left bottom)
+		)
+	)
+	(wire
+		(pts
+			(xy 707.39 572.77) (xy 690 572.77)
+		)
+		(stroke
+			(width 0)
+			(type default)
+		)
+	)
+	(wire
+		(pts
+			(xy 690 565.15) (xy 690 560.07)
+		)
+		(stroke
+			(width 0)
+			(type default)
+		)
+	)
+	(label "GND"
+		(at 690 560.07 0)
+		(effects
+			(font
+				(size 1.27 1.27)
+			)
+			(justify left bottom)
+		)
+	)
+	(no_connect
+		(at 707.39 631.19)
+	)
 	(sheet_instances
