File: dev_board.kicad_sch (KiCad schematic)
At the start: 177 parts, among them IC1 AD9609BCPZRL7-80, IC10 MP4541GN-Z, IC2 ENS161-BLGT_LGA9_T&R_1k5, IC3 ICM-42670-P, IC4 IWRL6432BDBAAMFR, IC5 MP4541GN-Z, IC6 THS8136IPHPR, IC7 TPS40304ADRCR, IC8 XCC1352R1F3RGZR, IC9 TPS40304ADRCR, J10 RJ45 / 8P8C LED, J11 SMA_RF_LAUNCH, J12 RP2350 USB PROGRAM, J13 DNP / not used, J14 DNP / not used, J15 IWRL USB PROGRAM, J2 Conn_02x26_Odd_Even, J4 SM03B-SRSS-TB, J5 STM32H7 GPIO/Fabric Breakout A, J6 STM32H7 GPIO/Fabric Breakout B, J9 HS/IWRL Fabric Breakout, SW1 SW_Push, SW2 SW_Push, U1 RP2350_80QFN, U2 LPS22HH, U3 STM32H750VBTx, U4 LAN8742A, U5 PGA113, U6 MCP6D11T-E/MS, U7 FT232RNL-TUBE, Y1 ABM8-272-T3

Commit message: more pcb stuff
Parts:
- removed R51: 0R/DNP, Resistor_SMD:R_0402_1005Metric, symbol Device:R
- added C96, C97, C98: 100p, Capacitor_SMD:C_0402_1005Metric, symbol Device:C
- added FL1: 0900PC15A0036, Package_LGA:Rohm_MLGA010V020A_LGA-10_2x2mm_P0.45mm_LayoutBorder2x3y, symbol 0900PC15A0036:0900PC15A0036
- added U8: XMSSJJ3G0PA-054, Package_TO_SOT_SMD:SOT-363_SC-70-6, symbol XMSSJJ3G0PA-054:XMSSJJ3G0PA-054
- added Y2: XRCMD48M000F1P2AR0, Crystal:Crystal_SMD_2016-4Pin_2.0x1.6mm, symbol Device:Crystal_GND24
Connections:
- net +1V1: no longer J2.43 (Pin_43), J4.3 (Pin_3)
- net +3V3: now also FL1.1 (ANT_2G4), U8.3 (PORT2), U8.4 (VDD)
- net CC_DIO_30: now also C97.2, FL1.4 (ANT_SUBG), U8.6 (CTL)
- net CC_DIO_6: now also IC2.7 (CSN)
- net CC_DIO_7: now also IC3.9 (INT2)
- net GND: now also J11.2 (Ext), C98.1, FL1.10 (GND), FL1.2 (GND), FL1.3 (GND), U8.2 (GND), Y2.2, Y2.4; no longer J13.5 (GND), J14.5 (GND)
- net GPIO6: no longer IC2.7 (CSN)
- net RP_SWCLK: no longer L1.2, U1.33 (SWCLK), U1.63 (VREG_LX)
- net VIN_RAW: no longer J14.1 (VBUS)
- net at J11.1 (In): now also C96.1
- net at IC8.5 (RX_TX): now also FL1.5 (RX_TX)
- net ADC_MODE_OR: no longer names the net of IC1.23 (MODE/OR)
- net CC_PROG_USB_D+: no longer names the net of J14.3 (D+)
- net CC_PROG_USB_D-: no longer names the net of J14.2 (D-)
- net CC_PROG_USB_VBUS: no longer names the net of J14.4 (ID)
- net CC_RF_N_2G4: no longer names the net of IC8.2 (RF_N_2_4GHZ)
- net CC_RF_N_2G4: now also FL1.8 (RF_N_2G4)
- net CC_RF_N_SUBG: no longer names the net of IC8.4 (RF_N_SUB_1GHZ)
- net CC_RF_N_SUBG: now also FL1.6 (RF_N_SUBG)
- net CC_RF_P_2G4: no longer names the net of IC8.1 (RF_P_2_4GHZ)
- net CC_RF_P_2G4: now also C98.2, FL1.9 (RF_P_2G4)
- net CC_RF_P_SUBG: no longer names the net of IC8.3 (RF_P_SUB_1GHZ)
- net CC_RF_P_SUBG: now also FL1.7 (RF_P_SUBG)
- net CC_X32K_Q1: no longer names the net of IC8.6 (X32K_Q1)
- net CC_X32K_Q2: no longer names the net of IC8.7 (X32K_Q2)
- net CC_X48M_N: no longer names the net of IC8.46 (X48M_N)
- net CC_X48M_N: now also Y2.3
- net CC_X48M_P: no longer names the net of IC8.47 (X48M_P)
- net CC_X48M_P: now also Y2.1
- net ETH_CT1: no longer names the net of J10.5 (CT2)
- net ETH_CT2: no longer names the net of J10.4 (CT1)
- net ETH_RXER: no longer names the net of U4.10 (RXER/PHYAD0)
- net IMU_AD0: no longer names the net of IC3.1 (AP_SDO_/_AP_AD0)
- net PHY_XTAL1: no longer names the net of U4.5 (XTAL1/CLKIN)
- net PHY_XTAL2: no longer names the net of U4.4 (XTAL2)
- net QSPI_SCLK: no longer names the net of U1.71 (QSPI_SCLK)
- net QSPI_SD0: no longer names the net of U1.72 (QSPI_SD0)
- net QSPI_SD1: no longer names the net of U1.74 (QSPI_SD1)
- net QSPI_SD2: no longer names the net of U1.73 (QSPI_SD2)
- net QSPI_SD3: no longer names the net of U1.70 (QSPI_SD3)
- net STM_USB_FS_DM: no longer names the net of J13.2 (D-)
- net STM_USB_FS_DP: no longer names the net of J13.3 (D+)
- net STM_USB_VBUS: no longer names the net of J13.1 (VBUS)
- net STM_VCAP_A: no longer names the net of U3.12 (PH0)
- new net: C96.2, U8.5 (RFC)
- new net: L1.2, U1.63 (VREG_LX)
- new net: C97.1, U8.1 (PORT1)
- new net RP_SWDIO: J2.43 (Pin_43), J4.3 (Pin_3)
- new net VREG_LX: U1.33 (SWCLK)
- no-connect marks 15 -> 39
Other:
- moved on the sheet: J11
