File: dev_board.kicad_pcb (KiCad board)
At the start: 4 copper layers, 100 x 50 mm, 176 parts, among them IC1 AD9609BCPZRL7-80, IC10 MP4541GN-Z, IC2 ENS161-BLGT_LGA9_T&R_1k5, IC3 ICM-42670-P, IC4 IWRL6432BDBAAMFR, IC5 MP4541GN-Z, IC6 THS8136IPHPR, IC7 TPS40304ADRCR, IC8 XCC1352R1F3RGZR, IC9 TPS40304ADRCR, J10 RJ45 / 8P8C LED, J11 SMA_RF_LAUNCH, J12 RP2350 USB PROGRAM, J13 DNP / not used, J14 DNP / not used, J15 IWRL USB PROGRAM, J2 Conn_02x26_Odd_Even, J4 SM03B-SRSS-TB, J5 STM32H7 GPIO/Fabric Breakout A, J6 STM32H7 GPIO/Fabric Breakout B, J9 HS/IWRL Fabric Breakout, SW1 SW_Push, SW2 SW_Push, U1 RP2350_80QFN, U2 LPS22HH, U3 STM32H750VBTx, U4 LAN8742A, U5 PGA113, U6 MCP6D11T-E/MS, U7 FT232RNL-TUBE, Y1 ABM8-272-T3

Commit message: more pcb stuff
Parts:
- added C95: 47n, Capacitor_SMD:C_0402_1005Metric, F.Cu at (-5.69, 29.2)
- J10: footprint Connector_RJ:RJ45_Amphenol_RJMG1BD3B8K1ANR -> Connector_RJ:RJ45_Wuerth_7499010211A_Horizontal
- moved R13 89.5 mm to (10.8, 35.6), turned to 90 degrees
- moved C87 81.1 mm to (89.6, 18.4), turned to 0 degrees
- moved R28 74.7 mm to (74.1, 8.84)
- moved C53 65.2 mm to (71.1, 14.1), turned to 180 degrees
- moved R38 65.1 mm to (81.1, 5.95)
- moved C54 63.9 mm to (71.2, 13.1), turned to 180 degrees
- moved R45 48.9 mm to (53.3, 43.6), turned to 90 degrees
- moved R29 48.7 mm to (52.9, 28.5), turned to 180 degrees
- moved R31 47.7 mm to (55.5, 35.8)
- moved C66 43.8 mm to (55.0, 45.4), turned to 180 degrees
- moved R48 42.2 mm to (52.6, 41.7), turned to -90 degrees
- moved R30 40.0 mm to (45.6, 36.6)
- moved R49 39.1 mm to (52.2, 38.5), turned to 180 degrees
- moved C67 38.9 mm to (51.7, 46.8), turned to 180 degrees
- moved C89 33.1 mm to (46.0, 40.0), turned to 0 degrees
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Routing:
- net /PHY_LED1_REGOFF: track 0.00 -> 36.1 mm
- net /PHY_LED2_INTSEL: track 0.00 -> 34.8 mm, vias 0 -> 2
- net /ETH_RX_P: track 0.00 -> 27.5 mm
- net /ETH_TX_P: track 0.00 -> 18.2 mm
- net /ETH_TX_N: track 0.00 -> 16.0 mm
- net /ADC_VCM: track 0.00 -> 14.1 mm, vias 0 -> 2
- net /ETH_CT: track 0.00 -> 9.64 mm
- net /ADC_AVDD_1V8: track 0.00 -> 9.25 mm, vias 0 -> 3
- net /DAC_FSADJ: track 0.00 -> 8.87 mm
- net /RP_SWCLK: track 0.00 -> 8.83 mm
- net /ETH_RX_N: track 0.00 -> 8.60 mm
- net /MP_FB: track 0.00 -> 8.33 mm
- net /ADC_VIN_P: track 0.00 -> 7.51 mm
- net /TPS_COMP: track 0.00 -> 6.91 mm
- net Net-(U6-OUT-): track 0.00 -> 6.83 mm
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- added copper zone on In2.Cu, net GND
