File: power.kicad_sch (KiCad schematic)
At the start: 28 parts, among them J1 VIN_IN, J2 TP_EN_PG, J3 TP_SW_FB, U3 MIC28516T-E/PHA

Commit message: Select L1 = KYOCERA AVX LMLP07C7M1R0DTAS; add KiCad CI branch protection
- Add proper power-inductor footprint L_Kyocera_LMLP07C7_7.0x6.9mm
  (2.4x6.0 mm pads, 4.6 mm centre-to-centre) to replace the 0603
  L_TODO_SELECT_1uH_15Aplus placeholder for the MIC28516 buck output
  inductor (net /Power/SW -> +3V3). Land pattern derived from the LMLP07
  series; flagged in descr for datasheet verification before fab.
- Record the part in power.kicad_sch L1 (Value, Footprint, Datasheet,
  Manufacturer, MPN) and in the production BOM.
- Add .github/workflows/kicad-checks.yml: headless KiCad 9 DRC gate on the
  production board (required) plus informational working-board DRC and
  schematic ERC, on pull_request/push to main.
- Add .github/BRANCH_PROTECTION.md with the exact rule to require the DRC
  check on main.

Note: physically placing/rerouting the 7 mm inductor on the boards is not
included here — see follow-up.

Co-Authored-By: Claude Opus 4.8 <noreply@anthropic.com>
Claude-Session: https://claude.ai/code/session_0186Z8rzxmfg6xURJrUFb6p5
Parts:
- L1: value 1uH, Isat > 15A -> 1uH LMLP07C7M1R0DTAS, Idc 15A / Isat 20A; footprint Inductor_SMD:L_TODO_SELECT_1uH_15Aplus -> Inductor_SMD:L_Kyocera_LMLP07C7_7.0x6.9mm; MPN (none) -> LMLP07C7M1R0DTAS; Manufacturer (none) -> KYOCERA AVX
Changed lines of the file:
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@@
 			)
 		)
-		(property "Value" "1uH, Isat > 15A"
+		(property "Value" "1uH LMLP07C7M1R0DTAS, Idc 15A / Isat 20A"
 			(at 157.21 69.21 0)
 			(effects
@@
 			)
 		)
-		(property "Footprint" "Inductor_SMD:L_TODO_SELECT_1uH_15Aplus"
+		(property "Footprint" "Inductor_SMD:L_Kyocera_LMLP07C7_7.0x6.9mm"
 			(at 157.21 66.67 0)
 			(effects
@@
 			)
 		)
-		(property "Datasheet" ""
+		(property "Datasheet" "https://datasheets.kyocera-avx.com/LMLPC.pdf"
 			(at 157.21 66.67 0)
 			(effects
@@
 			)
 		)
-		(property "Description" ""
+		(property "Description" "1uH power inductor, Idc 15A, Isat 20A, DCR ~6.1mOhm, shielded metal-alloy"
 			(at 157.21 66.67 0)
 			(effects
@@
 					(size 1.27 1.27)
 				)
+				(hide yes)
 			)
 		)
+		(property "Manufacturer" "KYOCERA AVX"
+			(at 157.21 66.67 0)
+			(effects
+				(font
+					(size 1.27 1.27)
+				)
+				(hide yes)
+			)
+		)
+		(property "MPN" "LMLP07C7M1R0DTAS"
+			(at 157.21 66.67 0)
+			(effects
+				(font
+					(size 1.27 1.27)
+				)
+				(hide yes)
+			)
+		)

Commit message: Correct LMLP07C7 land pattern to datasheet-verified dimensions
Replace the estimate-based footprint with one built from the actual
LMLP07C7 dimensional table in datasheets.kyocera-avx.com/LMLPD.pdf
(Style D, case 07C7): body 7.3x6.6mm (was estimated 7.0x6.9mm), pads
2.95x3.5mm at 5.45mm pitch (was estimated 2.4x6.0mm at 5.45mm pitch).
Also confirms LMLP07C7M1R0DTAS electricals: 1uH +/-20%, DCR 6.1/6.5
mOhm typ/max, IDC 15A typ, Isat 20A typ - matching the values already
used in the schematic/BOM.

Co-Authored-By: Claude Opus 4.8 <noreply@anthropic.com>
Claude-Session: https://claude.ai/code/session_0186Z8rzxmfg6xURJrUFb6p5
Parts:
- L1: footprint Inductor_SMD:L_Kyocera_LMLP07C7_7.0x6.9mm -> Inductor_SMD:L_Kyocera_LMLP07C7D_7.3x6.6mm
Changed lines of the file:
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@@
 			)
 		)
-		(property "Footprint" "Inductor_SMD:L_Kyocera_LMLP07C7_7.0x6.9mm"
+		(property "Footprint" "Inductor_SMD:L_Kyocera_LMLP07C7D_7.3x6.6mm"
 			(at 157.21 66.67 0)
 			(effects
