File: dev-real.kicad_pcb (KiCad board)
At the start: 4 copper layers, 105 x 105 mm, 318 parts, among them IC1 ICM-42670-P, IC2 ENS161-BLGT_LGA9_T&R_1k5, J1 VIN_IN, J10 USB-C USB2 DEBUG, J11 ARM_JTAG_10, J12 SOP0_SELECT, J13 SOP1_SELECT, J14 Conn_01x03, J15 Conn_01x03, J16 ARM_JTAG_10, J17 USB-C Receptacle USB2, J18 Conn_01x03_Pin, J19 Cortex SWD/JTAG, J2 TP_EN_PG, J20 USB-C USB2 DEVICE, J21 HR911105A MAGJACK, J22 Conn_02x10_Counter_Clockwise, J23 Conn_02x04_Odd_Even, J3 TP_SW_FB, J4 USB-C Receptacle USB2, J5 Conn_01x03_Pin, J6 ARM_Cortex_Debug_10, J7 SMA_ANT_50OHM, J8 3V3_IN, U1 MMC5633NJL, U10 USBLC6-2P6, U11 FT230XS-R, U12 FT230XS-R, U13 IWRL6432BDBAAMFR, U14 MX25R1635FZUIH0, U15 MX25R1635FZUIH0, U16 AMS1117-1.8, U17 THS8136, U18 MM8108-MF15457, U19 AP2112K-1.8, U2 LPS22HH, U20 PGA113AIDGSR, U21 AD9609BCPZRL7-80, U22 MCP6D11T-E/MS, U23 STM32H7S3Z8T6, U24 LAN8742A-CZ-TR, U25 USBLC6-2SC6, U3 MIC28516T-E/PHA, U4 RP2350B, U5 XCC1352R1F3RGZR, U6 XMSSJJ3G0PA-054, U7 TLV75518PDBV, U8 TLV75518PDBVR, U9 USBLC6-2P6, Y1 12MHz ABM8-272-T3, Y2 48MHz, Y3 40MHz, Y4 40MHz, Y5 24MHz, Y6 32.768kHz, Y7 25MHz

Commit message: Widen L1-area SW/+3V3 traces for 15A current capacity
Per-segment clearance-checked widening (0.2-0.4mm, up from 0.1-0.2mm)
of the /Power/SW and +3V3 track segments in the L1 reroute area,
matching the board's existing convention for local high-current power
hops. Verified via real kicad-cli DRC on both boards: 0 unconnected
items, no new violations (production: 1 pre-existing courtyard
overlap remains; working copy: unchanged 4 violations/6 unconnected,
all pre-existing and unrelated to L1).

Co-Authored-By: Claude Sonnet 5 <noreply@anthropic.com>
Claude-Session: https://claude.ai/code/session_0186Z8rzxmfg6xURJrUFb6p5
Parts:
- L1: value 1uH, Isat > 15A -> 1uH LMLP07C7M1R0DTAS, Idc 15A / Isat 20A; footprint Inductor_SMD:L_TODO_SELECT_1uH_15Aplus -> L_Kyocera_LMLP07C7D_7.3x6.6mm
- moved COUT2 1.85 mm to (68.9, 60.7)
Routing:
- net /Power/EXTVDD: track 18.5 -> 27.7 mm, vias 2 -> 6
- net /Power/EN: track 46.7 -> 52.4 mm, vias 8 -> 9
- net +3V3: track 495.6 -> 498.6 mm, vias 177 -> 178
- net GND: track 1636.9 -> 1639.7 mm, vias 356 -> 355
- net /RP2350/GPIO37: track 52.2 -> 54.5 mm, vias 2 -> 5
- net /Power/SW: track 91.0 -> 93.0 mm, vias 14 -> 15
- net /Power/PVDD: track 43.6 -> 45.5 mm, vias 5 -> 6
- net /IWRL6432BD/GPIO_5: track 88.9 -> 90.5 mm
- net /Power/FB: track 161.5 -> 160.0 mm
- net /AD9609/SCOPE_DRIVER_PD_N: track 156.8 -> 158.2 mm, vias 17 -> 19

Commit message: Fix C5/COUT2 courtyard overlap and widen remaining thin high-current traces
C5 relocated from (68.5,59.5) to (67.7,57.75)mm to clear its courtyard
overlap with COUT2 (COUT2 itself can't move - the channel to L1 is too
narrow in any orientation). Its two local nets (RIPPLE_INJ, FB) were
rerouted to the new pad positions, routing FB around an EXTVDD track
that blocked the direct path. Six duplicate FB stub segments left over
from earlier fix attempts this session were deduped in the process.

Production board DRC is now fully clean: 0 violations, 0 unconnected.

Also widened 5 thin (0.15mm) inner-layer segments on
/IWRL6432BD/USB_VBUS (found via a whole-board high-current trace
audit) to 0.2-0.3mm; two short segments near a neighboring via stay
at 0.15mm since widening them trips real clearance, documented in
PRODUCTION_HANDOFF.md as a follow-up item.

Working copy (dev-real.kicad_pcb) drops from 4 violations/6
unconnected to 3 violations/6 unconnected - the courtyard fix applied
there too; remaining items are pre-existing invalid_outline/BGA-area
issues unrelated to this work.

Co-Authored-By: Claude Sonnet 5 <noreply@anthropic.com>
Claude-Session: https://claude.ai/code/session_0186Z8rzxmfg6xURJrUFb6p5
Parts:
- moved C5 1.92 mm to (67.7, 57.8)
Routing:
- net /Power/FB: track 160.0 -> 166.3 mm
- net /Power/RIPPLE_INJ: track 10.8 -> 9.15 mm
Changed lines of the file:
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@@
 	(footprint "Capacitor_SMD:C_0603_1608Metric"
 		(layer "F.Cu")
-		(at 68.5 59.5)
+		(at 67.7 57.75)
 		(descr "Capacitor SMD 0603 (1608 Metric), square (rectangular) end terminal, IPC-7351 nominal, (Body size source: IPC-SM-782 page 76, https://www.pcb-3d.com/wordpress/wp-content/uploads/ipc-sm-782a_amendment_1_and_2.pdf), generated with kicad-footprint-generator")
 		(tags "capacitor")
@@
 	)
 	(segment
-		(start 71.7 73.35)
-		(end 69 73.35)
-		(width 0.2)
-		(layer "F.Cu")
-		(net 6)
-	)
-	(segment
-		(start 59.213 61.199999)
-		(end 59.25 61.199999)
+		(start 70.8 58.4)
+		(end 71 58.4)
 		(width 0.2)
 		(layer "F.Cu")
@@
 	)
 	(segment
-		(start 69.275 59.5)
-		(end 69.3 59.524999)
+		(start 71.7 73.35)
+		(end 69 73.35)
 		(width 0.2)
 		(layer "F.Cu")
@@
 	)
 	(segment
-		(start 63.985 62.25)
-		(end 64.2 62.25)
+		(start 71 58.4)
+		(end 71.6 59)
 		(width 0.2)
 		(layer "F.Cu")
@@
 	)
 	(segment
-		(start 69.275 59.5)
-		(end 69.3 59.524999)
+		(start 59.213 61.199999)
+		(end 59.25 61.199999)
 		(width 0.2)
 		(layer "F.Cu")
@@
 	)
 	(segment
-		(start 69.275 59.5)
-		(end 69.3 59.524999)
+		(start 63.985 62.25)
+		(end 64.2 62.25)
 		(width 0.2)
 		(layer "F.Cu")
@@
 	)
 	(segment
+		(start 69.2 59.6)
+		(end 69.3 59.524999)
+		(width 0.2)
+		(layer "F.Cu")
+		(net 6)
+	)
+	(segment
 		(start 99 94)
 		(end 99 93.45)
@@
 	)
 	(segment
+		(start 71 59.6)
+		(end 69.2 59.6)
+		(width 0.2)
+		(layer "F.Cu")
+		(net 6)
+	)
+	(segment
 		(start 66.899999 75.45)
 		(end 64.95 75.45)
@@
 	)
 	(segment
-		(start 69.275 59.5)
-		(end 69.3 59.524999)
+		(start 70.4 58)
+		(end 70.8 58.4)
 		(width 0.2)
 		(layer "F.Cu")
@@
 	)
 	(segment
+		(start 68.6 58)
+		(end 70.4 58)
+		(width 0.2)
+		(layer "F.Cu")
+		(net 6)
+	)
+	(segment
 		(start 62.5826 76.35)
 		(end 62.55 76.35)
@@
 	)
 	(segment
-		(start 58.1681 59.3431)
-		(end 58.5 59.675)
+		(start 71.6 59)
+		(end 71 59.6)
 		(width 0.2)
 		(layer "F.Cu")
@@
 	)
 	(segment
-		(start 90.45 84.45)
-		(end 90.75 84.75)
+		(start 58.1681 59.3431)
+		(end 58.5 59.675)
 		(width 0.2)
 		(layer "F.Cu")
@@
 	)
 	(segment
-		(start 69.275 59.5)
-		(end 69.3 59.524999)
+		(start 90.45 84.45)
+		(end 90.75 84.75)
 		(width 0.2)
 		(layer "F.Cu")
@@
 	)
 	(segment
-		(start 69.275 59.5)
-		(end 69.3 59.524999)
+		(start 68.475 57.75)
+		(end 68.6 58)
 		(width 0.2)
 		(layer "F.Cu")
@@
 	)
 	(segment
-		(start 67.725 59.5)
-		(end 65.674999 57.449999)
+		(start 60.325 55.6)
+		(end 62.075 53.85)
 		(width 0.2)
 		(layer "F.Cu")
@@
 	)
 	(segment
-		(start 60.325 55.6)
-		(end 62.075 53.85)
+		(start 66.925 57.75)
+		(end 65.674999 57.449999)
 		(width 0.2)
 		(layer "F.Cu")
@@
 		(start 52.6358 27.0538)
 		(end 52.6858 27.1038)
-		(width 0.15)
+		(width 0.25)
 		(layer "F.Cu")
 		(net 42)
@@
 		(start 60.535799 30.3038)
 		(end 60.9292 29.9128)
-		(width 0.15)
+		(width 0.2)
 		(layer "F.Cu")
 		(net 42)
@@
 		(start 51.0038 28.902)
 		(end 51.1038 28.752)
-		(width 0.25)
+		(width 0.3)
 		(layer "B.Cu")
 		(net 42)
@@
 		(start 57.2358 28.0038)
 		(end 57.4858 28.2538)
-		(width 0.15)
+		(width 0.3)
 		(layer "In2.Cu")
 		(net 42)
