File: XCC1352R1F3RGZR_breakout.kicad_sch (KiCad schematic)
At the start: 25 parts, among them J6 ARM_Cortex_Debug_10, J7 SMA_ANT_50OHM, U5 XCC1352R1F3RGZR, U6 XMSSJJ3G0PA-054, Y2 48MHz

Commit message: release: finalize dev-board fabrication package
- Remove two orphaned unannotated symbols (FB?, L?) from the XCC1352 sheet that crashed KiCad 9.0.7 ERC (access violation in eeschema.dll); they had no connections and no footprint counterparts on either PCB.

- Both dev-real.kicad_pcb and dev-real-production.kicad_pcb: 0 DRC errors, 0 unconnected items.

- Generate complete release/final/ with Gerbers, Excellon drills + maps, BOM, positions, schematic PDF, ERC/DRC reports, RELEASE_NOTES, SHA256 manifest.

/AD9609/SCOPE_BIAS remains the single user-accepted unresolved issue (no DC source; documented in RELEASE_NOTES).
Parts:
- removed FB?: BLM18HE152SN1, Inductor_SMD:L_0603_1608Metric, symbol Device:Ferrite_Bead
- removed L?: 6.8uH, Inductor_SMD:L_0603_1608Metric, symbol Device:L
Changed lines of the file:
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@@
-	)
-	(symbol
-		(lib_id "Device:Ferrite_Bead")
-		(at 35 90 0)
-		(unit 1)
-		(exclude_from_sim no)
-		(in_bom yes)
-		(on_board yes)
-		(dnp no)
-		(property "Reference" "FB?"
-			(at 35 85 0)
-			(effects
-				(font
-					(size 1.27 1.27)
-				)
-			)
-		)
-		(property "Value" "BLM18HE152SN1"
-			(at 35 95 0)
-			(effects
-				(font
-					(size 1.27 1.27)
-				)
-			)
-		)
-		(property "Footprint" "Inductor_SMD:L_0603_1608Metric"
-			(at 35 97 0)
-			(effects
-				(font
-					(size 1.27 1.27)
-				)
-				(hide yes)
-			)
-		)
-		(property "Datasheet" ""
-			(at 35 99 0)
-			(effects
-				(font
-					(size 1.27 1.27)
-				)
-				(hide yes)
-			)
-		)
-		(property "Description" ""
-			(at 35 90 0)
-			(effects
-				(font
-					(size 1.27 1.27)
-				)
-			)
-		)
-		(pin "1"
-		)
-		(pin "2"
-		)
-		(instances
-			(project "dev-real"
-				(path "/53d6bfbe-b600-4a9a-86be-e807ba51b147/e97ea36d-e095-4b7a-ba32-9f0d594e91b6"
-					(reference "FB?")
-					(unit 1)
-				)
-			)
-		)
 	)
 	(symbol
@@
 					(unit 1)
 				)
-			)
-		)
-	)
-	(symbol
-		(lib_id "Device:L")
-		(at 35 77 0)
-		(unit 1)
-		(exclude_from_sim no)
-		(in_bom yes)
-		(on_board yes)
-		(dnp no)
-		(property "Reference" "L?"
-			(at 35 72 0)
-			(effects
-				(font
-					(size 1.27 1.27)
-				)
-			)
-		)
-		(property "Value" "6.8uH"
-			(at 35 82 0)
-			(effects
-				(font
-					(size 1.27 1.27)
-				)
-			)
-		)
-		(property "Footprint" "Inductor_SMD:L_0603_1608Metric"
-			(at 35 84 0)
-			(effects
-				(font
-					(size 1.27 1.27)
-				)
-				(hide yes)
-			)
-		)
-		(property "Datasheet" ""
-			(at 35 86 0)
-			(effects
-				(font
-					(size 1.27 1.27)
-				)
-				(hide yes)
-			)
-		)
-		(property "Description" ""
-			(at 35 77 0)
-			(effects
-				(font
-					(size 1.27 1.27)
-				)
-			)
-		)
-		(pin "1"
-		)
-		(pin "2"
-		)
-		(instances
-			(project "dev-real"
-				(path "/53d6bfbe-b600-4a9a-86be-e807ba51b147/e97ea36d-e095-4b7a-ba32-9f0d594e91b6"
-					(reference "L?")
-					(unit 1)
-				)
